Commit message: V031: 修掉 left_hip_yaw_link 与右侧差 10.3 g 的质量不对称
对称性体检里唯一量级超过 1 g 的左右差异：left_hip_yaw_link 质量
0.323365 kg，right_hip_yaw_link 0.333676 kg，差 10.311 g（3.09%），
左腿整链 1.063113 / 右腿 1.073424 kg（0.961%）。其余连杆质量差为 0。

改动：把左侧质量改成与右侧同值 0.333676（URDF 里写全精度
0.333676134224531），三处同步——URDF（easymjcf 的上游真源）、
mjcf/pikachu_v031.xml（easymjcf 直出）、mjcf/pikachu_v031_train.xml
（build_v031_train_xml.py 从后者文本生成，重新生成后 diff 只有这一行）。
整机质量 6.759964 → 6.770275 kg（+10.311 g，+0.153%）。

未改动的残留：该连杆质心镜像残差仍有 0.580 mm、惯量张量相对差 0.51%
（hip_pitch_link 0.068 mm、knee_up_link 0.35%），这些是左右两件 CAD
零件的固有差别，未按镜像强改——只统一了用户要求的质量项。

复验：scripts/diag_v031_symmetry.py 第 1 节所有 dm(g) 归零；第 5 节
20 组随机驱动配置下整机镜像残差仍是位置 0.000000000 mm / 姿态 0.000e+00，
说明本次改动没有破坏原有的严格镜像运动学。

注意：本改动落盘时 T6 档已在跑（进程启动时已加载旧模型），
Sym/SymClip/Clip/YawHuber 四档会加载修复后的模型。

Co-Authored-By: Claude Code <noreply@anthropic.com>

File: src/mjlab/asset_zoo/robots/pikachu/xmls/pikachu_v031/urdf/pikachu_v031.urdf (robot description, URDF)
Before this commit: robot pikachu_v032, 15 links, 14 joints
Links:
- link left_hip_yaw_link: mass 0.323365494488295 -> 0.333676134224531
